Commit message: Added vrep package

File: thymioid/models/thymioid.urdf.xacro (robot description, xacro)
@@ -54,10 +54,10 @@
   </joint>
   <joint name="camera_body_support_joint" type="fixed">
-    <origin xyz="0.015 0 0" rpy="0 0 0"/>
+    <origin xyz="0.015 0 0" rpy="0 0.2618 0"/>
     <parent link="camera_support_link"/>
     <child link="camera_body_link"/>
   </joint>
   <joint name="camera_frame_joint" type="fixed">
-    <origin xyz="0.0 0 0" rpy="0 0 0"/>
+    <origin xyz="0.0 0 0" rpy="-1.5708 0 -1.5708"/>
     <parent link="camera_body_link"/>
     <child link="camera_link"/>

Commit message: Minor changes

File: thymioid/models/thymioid.urdf.xacro (robot description, xacro)
@@ -36,5 +36,5 @@
     <visual>
       <geometry>
-	<box size="0.016 0.02 0.01"/>
+	<box size="0.02 0.01 0.016"/>
       </geometry>
       <material name="Grey">
@@ -59,5 +59,5 @@
   </joint>
   <joint name="camera_frame_joint" type="fixed">
-    <origin xyz="0.0 0 0" rpy="0 0 0"/>
+    <origin xyz="0.0 0 0" rpy="-1.5708 0 -1.5708"/>
     <parent link="camera_body_link"/>
     <child link="camera_link"/>
