Commit message: Copied distortion model from real camera

File: thymioid_description/urdf/camera.urdf.xacro (robot description, xacro)
@@ -6,14 +6,10 @@
         <origin xyz="0 0 0"/>
         <mass value="0.01"/>
-        <inertia ixx="1e-3" ixy="0" ixz="0" iyy="1e-3" iyz="0" izz="1e-3"/>
+        <inertia ixx="1e-6" ixy="0" ixz="0" iyy="1e-6" iyz="0" izz="1e-6"/>
       </inertial>
-      <collision>
-        <geometry>
-           <mesh filename="package://thymioid_description/meshes/camera_support.dae" />
-        </geometry>
-      </collision>
+      <!-- <collision> <geometry> <mesh filename="package://thymioid_description/meshes/camera_support.dae" /> </geometry> </collision> -->
       <visual>
         <geometry>
-  	       <mesh filename="package://thymioid_description/meshes/camera_support.dae" />
+          <mesh filename="package://thymioid_description/meshes/camera_support.dae"/>
         </geometry>
       </visual>
@@ -21,41 +17,21 @@
     <link name="camera_body_link">
       <inertial>
-        <origin xyz="0 0 0"/>
-        <mass value="0.01"/>
-        <inertia ixx="1e-3" ixy="0" ixz="0" iyy="1e-3" iyz="0" izz="1e-3"/>
+        <origin xyz="0.008 0 0"/>
+        <mass value="0.02"/>
+        <inertia ixx="6e-6" ixy="0" ixz="0" iyy="2e-6" iyz="0" izz="5e-6"/>
       </inertial>
       <collision>
         <geometry>
-           <mesh filename="package://thymioid_description/meshes/camera.dae" />
+          <mesh filename="package://thymioid_description/meshes/camera.dae"/>
         </geometry>
       </collision>
       <visual>
         <geometry>
-  	       <mesh filename="package://thymioid_description/meshes/camera.dae" />
+          <mesh filename="package://thymioid_description/meshes/camera.dae"/>
         </geometry>
       </visual>
     </link>
-    <link name="camera_link">
-      <!-- <inertial>
-        <origin xyz="0 0 0"/>
-        <mass value="0.01"/>
-        <inertia ixx="1e-3" ixy="0" ixz="0" iyy="1e-3" iyz="0" izz="1e-3"/>
-      </inertial>
-      <collision>
-        <geometry>
-           <box size="0.02 0.01 0.016"/>
-        </geometry>
-      </collision>
-      <visual>
-        <geometry>
-  	       <box size="0.02 0.01 0.016"/>
-        </geometry>
-        <material name="Grey">
-  	       <color rgba="0.0 0.0 0.0 1.0"/>
-        </material>
-      </visual> -->
-    </link>
-    <link name="camera_optical_link">
-    </link>
+    <link name="camera_link"/>
+    <link name="camera_optical_link"/>
     <joint name="ups_camera_joint" type="fixed">
       <origin xyz="0.0047 -0.032 0.044" rpy="0 0 0"/>
@@ -70,5 +46,5 @@
       <limit lower="-0.7" upper="0.9" effort="0" velocity="0"/>
     </joint>
-<!-- http://www.ros.org/reps/rep-0103.html -->
+    <!-- http://www.ros.org/reps/rep-0103.html -->
     <joint name="camera_frame_joint" type="fixed">
       <origin xyz="0.01 0 0"/>
@@ -82,8 +58,8 @@
     </joint>
     <gazebo reference="camera_link">
-      <sensor type="camera" name="camera1">
+      <sensor type="camera" name="head_camera">
         <update_rate>30.0</update_rate>
-        <camera name="head">
-          <horizontal_fov>1.3962634</horizontal_fov>
+        <camera name="head_camera">
+          <horizontal_fov>0.786</horizontal_fov>
           <image>
             <width>640</width>
@@ -92,6 +68,6 @@
           </image>
           <clip>
-            <near>0.02</near>
-            <far>300</far>
+            <near>0.01</near>
+            <far>20</far>
           </clip>
           <noise>
@@ -108,10 +84,13 @@
           <cameraInfoTopicName>camera_info</cameraInfoTopicName>
           <frameName>camera_optical_link</frameName>
-          <hackBaseline>0.07</hackBaseline>
-          <distortionK1>0.0</distortionK1>
-          <distortionK2>0.0</distortionK2>
-          <distortionK3>0.0</distortionK3>
-          <distortionT1>0.0</distortionT1>
+          <hackBaseline>0.0</hackBaseline>
+          <distortionK1>-0.003061</distortionK1>
+          <distortionK2>0.044691</distortionK2>
+          <distortionK3>0.012541</distortionK3>
+          <distortionT1>-0.00085</distortionT1>
           <distortionT2>0.0</distortionT2>
+          <CxPrime>333.88</CxPrime>
+          <Cx>334.87</Cx>
+          <Cy>281.10</Cy>
         </plugin>
       </sensor>

Commit message: Added (optional) control to change camera pitch

File: thymioid_description/urdf/camera.urdf.xacro (robot description, xacro)
@@ -1,5 +1,7 @@
 <?xml version="1.0"?>
 <robot xmlns:xacro="http://playerstage.sourceforge.net/gazebo/xmlschema/#xacro">
-  <xacro:macro name="web_camera">
+  <xacro:arg name="camera_joint_type" default="fixed"/>
+  <xacro:arg name="camera_pitch" default="0"/>
+  <xacro:macro name="web_camera" params="camera_joint_type camera_pitch">
     <link name="camera_support_link">
       <inertial>
@@ -39,10 +41,11 @@
       <child link="camera_support_link"/>
     </joint>
-    <joint name="camera_body_support_joint" type="fixed">
-      <origin xyz="0.0095 0 -0.0051" rpy="0 0.2618 0"/>
+    <joint name="camera_body_support_joint" type="$(arg camera_joint_type)">
+      <origin xyz="0.0095 0 -0.0051" rpy="0 $(arg camera_pitch) 0"/>
       <parent link="camera_support_link"/>
       <child link="camera_body_link"/>
       <axis xyz="0 1 0"/>
-      <limit lower="-0.7" upper="0.9" effort="0" velocity="0"/>
+      <limit lower="-0.34" upper="1.3" effort="1e-9" velocity="1e-9"/>
+      <dynamics friction="1e6"/>
     </joint>
     <!-- http://www.ros.org/reps/rep-0103.html -->

File: thymioid_description/urdf/thymioid.urdf.xacro (robot description, xacro)
@@ -117,4 +117,4 @@
     <child link="odroid_link"/>
   </joint>
-  <xacro:web_camera/>
+  <xacro:web_camera camera_joint_type="$(arg camera_joint_type)" camera_pitch="$(arg camera_pitch)"/>
 </robot>

Commit message: Tested

File: thymioid_description/urdf/camera.urdf.xacro (robot description, xacro)
@@ -46,5 +46,5 @@
       <child link="camera_body_link"/>
       <axis xyz="0 1 0"/>
-      <limit lower="-0.34" upper="1.3" effort="1e-9" velocity="1e-9"/>
+      <limit lower="-0.35" upper="1.31" effort="1e-9" velocity="1e-9"/>
       <dynamics friction="1e6"/>
     </joint>

Commit message: Added camera_is_on option

File: thymioid_description/urdf/camera.urdf.xacro (robot description, xacro)
@@ -3,5 +3,6 @@
   <xacro:arg name="camera_joint_type" default="fixed"/>
   <xacro:arg name="camera_pitch" default="0"/>
-  <xacro:macro name="web_camera" params="camera_joint_type camera_pitch">
+  <xacro:arg name="camera_is_on" default="true"/>
+  <xacro:macro name="web_camera" params="camera_joint_type camera_pitch camera_is_on">
     <link name="camera_support_link">
       <inertial>
@@ -60,43 +61,45 @@
       <child link="camera_optical_link"/>
     </joint>
-    <gazebo reference="camera_link">
-      <sensor type="camera" name="head_camera">
-        <update_rate>30.0</update_rate>
-        <camera name="head_camera">
-          <horizontal_fov>0.786</horizontal_fov>
-          <image>
-            <width>640</width>
-            <height>480</height>
-            <format>R8G8B8</format>
-          </image>
-          <clip>
-            <near>0.01</near>
-            <far>20</far>
-          </clip>
-          <noise>
-            <type>gaussian</type>
-            <mean>0.0</mean>
-            <stddev>0.007</stddev>
-          </noise>
-        </camera>
-        <plugin name="camera_controller" filename="libgazebo_ros_camera.so">
-          <alwaysOn>true</alwaysOn>
-          <updateRate>0.0</updateRate>
-          <cameraName>camera</cameraName>
-          <imageTopicName>image_raw</imageTopicName>
-          <cameraInfoTopicName>camera_info</cameraInfoTopicName>
-          <frameName>camera_optical_link</frameName>
-          <hackBaseline>0.0</hackBaseline>
-          <distortionK1>-0.003061</distortionK1>
-          <distortionK2>0.044691</distortionK2>
-          <distortionK3>0.012541</distortionK3>
-          <distortionT1>-0.00085</distortionT1>
-          <distortionT2>0.0</distortionT2>
-          <CxPrime>333.88</CxPrime>
-          <Cx>334.87</Cx>
-          <Cy>281.10</Cy>
-        </plugin>
-      </sensor>
-    </gazebo>
+    <xacro:if value="$(arg camera_is_on)">
+      <gazebo reference="camera_link">
+        <sensor type="camera" name="head_camera">
+          <update_rate>30.0</update_rate>
+          <camera name="head_camera">
+            <horizontal_fov>0.786</horizontal_fov>
+            <image>
+              <width>640</width>
+              <height>480</height>
+              <format>R8G8B8</format>
+            </image>
+            <clip>
+              <near>0.01</near>
+              <far>20</far>
+            </clip>
+            <noise>
+              <type>gaussian</type>
+              <mean>0.0</mean>
+              <stddev>0.007</stddev>
+            </noise>
+          </camera>
+          <plugin name="camera_controller" filename="libgazebo_ros_camera.so">
+            <alwaysOn>true</alwaysOn>
+            <updateRate>0.0</updateRate>
+            <cameraName>camera</cameraName>
+            <imageTopicName>image_raw</imageTopicName>
+            <cameraInfoTopicName>camera_info</cameraInfoTopicName>
+            <frameName>camera_optical_link</frameName>
+            <hackBaseline>0.0</hackBaseline>
+            <distortionK1>-0.003061</distortionK1>
+            <distortionK2>0.044691</distortionK2>
+            <distortionK3>0.012541</distortionK3>
+            <distortionT1>-0.00085</distortionT1>
+            <distortionT2>0.0</distortionT2>
+            <CxPrime>333.88</CxPrime>
+            <Cx>334.87</Cx>
+            <Cy>281.10</Cy>
+          </plugin>
+        </sensor>
+      </gazebo>
+    </xacro:if>
   </xacro:macro>
 </robot>

File: thymioid_description/urdf/thymioid.urdf.xacro (robot description, xacro)
@@ -117,4 +117,5 @@
     <child link="odroid_link"/>
   </joint>
-  <xacro:web_camera camera_joint_type="$(arg camera_joint_type)" camera_pitch="$(arg camera_pitch)"/>
+  <xacro:web_camera camera_joint_type="$(arg camera_joint_type)" camera_pitch="$(arg camera_pitch)"
+    camera_is_on="$(arg camera_is_on)"/>
 </robot>

Commit message: Cleaned up

File: thymioid_description/urdf/camera.urdf.xacro (robot description, xacro)
@@ -1,8 +1,6 @@
 <?xml version="1.0"?>
 <robot xmlns:xacro="http://playerstage.sourceforge.net/gazebo/xmlschema/#xacro">
-  <xacro:arg name="camera_joint_type" default="fixed"/>
-  <xacro:arg name="camera_pitch" default="0"/>
-  <xacro:macro name="web_camera" params="camera_joint_type camera_pitch">
-    <link name="camera_support_link">
+  <xacro:macro name="web_camera" params="tf_prefix='' camera_joint_type='fixed' camera_pitch=0">
+    <link name="${tf_prefix}camera_support_link">
       <inertial>
         <origin xyz="0 0 0"/>
@@ -17,5 +15,5 @@
       </visual>
     </link>
-    <link name="camera_body_link">
+    <link name="${tf_prefix}camera_body_link">
       <inertial>
         <origin xyz="0.008 0 0"/>
@@ -34,15 +32,15 @@
       </visual>
     </link>
-    <link name="camera_link"/>
-    <link name="camera_optical_link"/>
-    <joint name="ups_camera_joint" type="fixed">
+    <link name="${tf_prefix}camera_link"/>
+    <link name="${tf_prefix}camera_optical_link"/>
+    <joint name="${tf_prefix}ups_camera_joint" type="fixed">
       <origin xyz="0.0047 -0.032 0.044" rpy="0 0 0"/>
-      <parent link="ups_link"/>
-      <child link="camera_support_link"/>
+      <parent link="${tf_prefix}ups_link"/>
+      <child link="${tf_prefix}camera_support_link"/>
     </joint>
-    <joint name="camera_body_support_joint" type="$(arg camera_joint_type)">
+    <joint name="${tf_prefix}camera_body_support_joint" type="$(arg camera_joint_type)">
       <origin xyz="0.0095 0 -0.0051" rpy="0 $(arg camera_pitch) 0"/>
-      <parent link="camera_support_link"/>
-      <child link="camera_body_link"/>
+      <parent link="${tf_prefix}camera_support_link"/>
+      <child link="${tf_prefix}camera_body_link"/>
       <axis xyz="0 1 0"/>
       <limit lower="-0.34" upper="1.3" effort="1e-9" velocity="1e-9"/>
@@ -50,15 +48,15 @@
     </joint>
     <!-- http://www.ros.org/reps/rep-0103.html -->
-    <joint name="camera_frame_joint" type="fixed">
+    <joint name="${tf_prefix}camera_frame_joint" type="fixed">
       <origin xyz="0.01 0 0"/>
-      <parent link="camera_body_link"/>
-      <child link="camera_link"/>
+      <parent link="${tf_prefix}camera_body_link"/>
+      <child link="${tf_prefix}camera_link"/>
     </joint>
-    <joint name="camera_optical_joint" type="fixed">
+    <joint name="${tf_prefix}camera_optical_joint" type="fixed">
       <origin xyz="0 0 0" rpy="${-pi/2} 0 ${-pi/2}"/>
-      <parent link="camera_link"/>
-      <child link="camera_optical_link"/>
+      <parent link="${tf_prefix}camera_link"/>
+      <child link="${tf_prefix}camera_optical_link"/>
     </joint>
-    <gazebo reference="camera_link">
+    <gazebo reference="${tf_prefix}camera_link">
       <sensor type="camera" name="head_camera">
         <update_rate>30.0</update_rate>
@@ -103,5 +101,5 @@
           <!-- This makes the plugin segfault [tested on macos] -->
           <!-- <camera_name>camera</camera_name> -->
-          <frame_name>camera_optical_link</frame_name>
+          <frame_name>${tf_prefix}camera_optical_link</frame_name>
           <hack_baseline>0.0</hack_baseline>
         </plugin>

File: thymioid_description/urdf/thymioid.urdf.xacro (robot description, xacro)
@@ -1,9 +1,15 @@
 <?xml version="1.0"?>
 <robot name="thymioid" xmlns:xacro="http://playerstage.sourceforge.net/gazebo/xmlschema/#xacro">
-  <xacro:include filename="$(find thymio_description)/share/thymio_description/urdf/base.urdf.xacro"/>
+  <xacro:include filename="$(find thymio_description)/urdf/base.urdf.xacro"/>
   <xacro:include filename="camera.urdf.xacro"/>
   <xacro:arg name="power_pack" default="true"/>
   <xacro:thymio/>
-  <link name="chassis_link">
+  <xacro:if value="${_name != ''}">
+    <xacro:property name="tf_prefix" value="${_name}/"/>
+  </xacro:if>
+  <xacro:if value="${_name == ''}">
+    <xacro:property name="tf_prefix" value=""/>
+  </xacro:if>
+  <link name="${tf_prefix}chassis_link">
     <inertial>
       <origin xyz="0 0 0"/>
@@ -22,10 +28,10 @@
     </visual>
   </link>
-  <joint name="base_chassis_joint" type="fixed">
+  <joint name="${tf_prefix}base_chassis_joint" type="fixed">
     <origin xyz="0.0081 0 0.053" rpy="0 0 0"/>
-    <parent link="base_link"/>
-    <child link="chassis_link"/>
+    <parent link="${tf_prefix}base_link"/>
+    <child link="${tf_prefix}chassis_link"/>
   </joint>
-  <link name="spacers_link">
+  <link name="${tf_prefix}spacers_link">
     <inertial>
       <origin xyz="0 0 0"/>
@@ -44,11 +50,11 @@
     </visual>
   </link>
-  <joint name="chassis_spacers_joint" type="fixed">
+  <joint name="${tf_prefix}chassis_spacers_joint" type="fixed">
     <origin xyz="-0.016 0.041 0.0344" rpy="0 0 0"/>
-    <parent link="chassis_link"/>
-    <child link="spacers_link"/>
+    <parent link="${tf_prefix}chassis_link"/>
+    <child link="${tf_prefix}spacers_link"/>
   </joint>
   <xacro:if value="$(arg power_pack)">
-    <link name="power_pack_link">
+    <link name="${tf_prefix}power_pack_link">
       <inertial>
         <origin xyz="0 0 0"/>
@@ -67,11 +73,11 @@
       </visual>
     </link>
-    <joint name="base_power_pack_joint" type="fixed">
+    <joint name="${tf_prefix}base_power_pack_joint" type="fixed">
       <origin xyz="0 0 0.0143"/>
-      <parent link="chassis_link"/>
-      <child link="power_pack_link"/>
+      <parent link="${tf_prefix}chassis_link"/>
+      <child link="${tf_prefix}power_pack_link"/>
     </joint>
   </xacro:if>
-  <link name="ups_link">
+  <link name="${tf_prefix}ups_link">
     <inertial>
       <origin xyz="0.004 -0.03 0.024"/>
@@ -90,10 +96,10 @@
     </visual>
   </link>
-  <joint name="spacers_ups_joint" type="fixed">
+  <joint name="${tf_prefix}spacers_ups_joint" type="fixed">
     <origin xyz="0.031 0 0.0078" rpy="0 0 0"/>
-    <parent link="spacers_link"/>
-    <child link="ups_link"/>
+    <parent link="${tf_prefix}spacers_link"/>
+    <child link="${tf_prefix}ups_link"/>
   </joint>
-  <link name="odroid_link">
+  <link name="${tf_prefix}odroid_link">
     <inertial>
       <origin xyz="0.006 -0.045 0.022"/>
@@ -112,9 +118,9 @@
     </visual>
   </link>
-  <joint name="spacers_odroid_joint" type="fixed">
+  <joint name="${tf_prefix}spacers_odroid_joint" type="fixed">
     <origin xyz="0.01 0 0 " rpy="0 0 0"/>
-    <parent link="spacers_link"/>
-    <child link="odroid_link"/>
+    <parent link="${tf_prefix}spacers_link"/>
+    <child link="${tf_prefix}odroid_link"/>
   </joint>
-  <xacro:web_camera camera_joint_type="$(arg camera_joint_type)" camera_pitch="$(arg camera_pitch)"/>
+  <xacro:web_camera tf_prefix="${tf_prefix}" camera_joint_type="$(arg camera_joint_type)" camera_pitch="$(arg camera_pitch)"/>
 </robot>
