Commit message: Upgraded to ROS1 Noetic. Switched from implicit to explicit tf_prefix

File: thymioid_description/urdf/camera.urdf.xacro (robot description, xacro)
@@ -4,6 +4,6 @@
   <xacro:arg name="camera_pitch" default="0"/>
   <xacro:arg name="camera_is_on" default="true"/>
-  <xacro:macro name="web_camera" params="camera_joint_type camera_pitch camera_is_on">
-    <link name="camera_support_link">
+  <xacro:macro name="web_camera" params="camera_joint_type camera_pitch camera_is_on tf_prefix:=''">
+    <link name="${tf_prefix}camera_support_link">
       <inertial>
         <origin xyz="0 0 0"/>
@@ -18,5 +18,5 @@
       </visual>
     </link>
-    <link name="camera_body_link">
+    <link name="${tf_prefix}camera_body_link">
       <inertial>
         <origin xyz="0.008 0 0"/>
@@ -35,15 +35,15 @@
       </visual>
     </link>
-    <link name="camera_link"/>
-    <link name="camera_optical_link"/>
-    <joint name="ups_camera_joint" type="fixed">
+    <link name="${tf_prefix}camera_link"/>
+    <link name="${tf_prefix}camera_optical_link"/>
+    <joint name="${tf_prefix}ups_camera_joint" type="fixed">
       <origin xyz="0.0047 -0.032 0.044" rpy="0 0 0"/>
-      <parent link="ups_link"/>
-      <child link="camera_support_link"/>
+      <parent link="${tf_prefix}ups_link"/>
+      <child link="${tf_prefix}camera_support_link"/>
     </joint>
-    <joint name="camera_body_support_joint" type="$(arg camera_joint_type)">
+    <joint name="${tf_prefix}camera_body_support_joint" type="$(arg camera_joint_type)">
       <origin xyz="0.0095 0 -0.0051" rpy="0 $(arg camera_pitch) 0"/>
-      <parent link="camera_support_link"/>
-      <child link="camera_body_link"/>
+      <parent link="${tf_prefix}camera_support_link"/>
+      <child link="${tf_prefix}camera_body_link"/>
       <axis xyz="0 1 0"/>
       <limit lower="-0.35" upper="1.31" effort="1e-9" velocity="1e-9"/>
@@ -51,16 +51,16 @@
     </joint>
     <!-- http://www.ros.org/reps/rep-0103.html -->
-    <joint name="camera_frame_joint" type="fixed">
+    <joint name="${tf_prefix}camera_frame_joint" type="fixed">
       <origin xyz="0.01 0 0"/>
-      <parent link="camera_body_link"/>
-      <child link="camera_link"/>
+      <parent link="${tf_prefix}camera_body_link"/>
+      <child link="${tf_prefix}camera_link"/>
     </joint>
-    <joint name="camera_optical_joint" type="fixed">
+    <joint name="${tf_prefix}camera_optical_joint" type="fixed">
       <origin xyz="0 0 0" rpy="${-pi/2} 0 ${-pi/2}"/>
-      <parent link="camera_link"/>
-      <child link="camera_optical_link"/>
+      <parent link="${tf_prefix}camera_link"/>
+      <child link="${tf_prefix}camera_optical_link"/>
     </joint>
     <xacro:if value="$(arg camera_is_on)">
-      <gazebo reference="camera_link">
+      <gazebo reference="${tf_prefix}camera_link">
         <sensor type="camera" name="head_camera">
           <update_rate>30.0</update_rate>
@@ -88,5 +88,5 @@
             <imageTopicName>image_raw</imageTopicName>
             <cameraInfoTopicName>camera_info</cameraInfoTopicName>
-            <frameName>camera_optical_link</frameName>
+            <frameName>${tf_prefix}camera_optical_link</frameName>
             <hackBaseline>0.0</hackBaseline>
             <distortionK1>-0.003061</distortionK1>

File: thymioid_description/urdf/thymioid.urdf.xacro (robot description, xacro)
@@ -4,6 +4,14 @@
   <xacro:include filename="$(find thymioid_description)/urdf/camera.urdf.xacro"/>
   <xacro:arg name="power_pack" default="true"/>
+  <xacro:arg name="name" default=""/>
+  <xacro:property name="_name" value="$(arg name)"/>
+  <xacro:if value="${_name != ''}">
+    <xacro:property name="tf_prefix" value="${_name}/"/>
+  </xacro:if>
+  <xacro:if value="${_name == ''}">
+    <xacro:property name="tf_prefix" value=""/>
+  </xacro:if>
   <xacro:thymio/>
-  <link name="chassis_link">
+  <link name="${tf_prefix}chassis_link">
     <inertial>
       <origin xyz="0 0 0"/>
@@ -22,10 +30,10 @@
     </visual>
   </link>
-  <joint name="base_chassis_joint" type="fixed">
+  <joint name="${tf_prefix}base_chassis_joint" type="fixed">
     <origin xyz="0.0081 0 0.053" rpy="0 0 0"/>
-    <parent link="base_link"/>
-    <child link="chassis_link"/>
+    <parent link="${tf_prefix}base_link"/>
+    <child link="${tf_prefix}chassis_link"/>
   </joint>
-  <link name="spacers_link">
+  <link name="${tf_prefix}spacers_link">
     <inertial>
       <origin xyz="0 0 0"/>
@@ -44,11 +52,11 @@
     </visual>
   </link>
-  <joint name="chassis_spacers_joint" type="fixed">
+  <joint name="${tf_prefix}chassis_spacers_joint" type="fixed">
     <origin xyz="-0.016 0.041 0.0344" rpy="0 0 0"/>
-    <parent link="chassis_link"/>
-    <child link="spacers_link"/>
+    <parent link="${tf_prefix}chassis_link"/>
+    <child link="${tf_prefix}spacers_link"/>
   </joint>
   <xacro:if value="$(arg power_pack)">
-    <link name="power_pack_link">
+    <link name="${tf_prefix}power_pack_link">
       <inertial>
         <origin xyz="0 0 0"/>
@@ -67,11 +75,11 @@
       </visual>
     </link>
-    <joint name="base_power_pack_joint" type="fixed">
+    <joint name="${tf_prefix}base_power_pack_joint" type="fixed">
       <origin xyz="0 0 0.0143"/>
-      <parent link="chassis_link"/>
-      <child link="power_pack_link"/>
+      <parent link="${tf_prefix}chassis_link"/>
+      <child link="${tf_prefix}power_pack_link"/>
     </joint>
   </xacro:if>
-  <link name="ups_link">
+  <link name="${tf_prefix}ups_link">
     <inertial>
       <origin xyz="0.004 -0.03 0.024"/>
@@ -90,10 +98,10 @@
     </visual>
   </link>
-  <joint name="spacers_ups_joint" type="fixed">
+  <joint name="${tf_prefix}spacers_ups_joint" type="fixed">
     <origin xyz="0.031 0 0.0078" rpy="0 0 0"/>
-    <parent link="spacers_link"/>
-    <child link="ups_link"/>
+    <parent link="${tf_prefix}spacers_link"/>
+    <child link="${tf_prefix}ups_link"/>
   </joint>
-  <link name="odroid_link">
+  <link name="${tf_prefix}odroid_link">
     <inertial>
       <origin xyz="0.006 -0.045 0.022"/>
@@ -112,10 +120,10 @@
     </visual>
   </link>
-  <joint name="spacers_odroid_joint" type="fixed">
+  <joint name="${tf_prefix}spacers_odroid_joint" type="fixed">
     <origin xyz="0.01 0 0 " rpy="0 0 0"/>
-    <parent link="spacers_link"/>
-    <child link="odroid_link"/>
+    <parent link="${tf_prefix}spacers_link"/>
+    <child link="${tf_prefix}odroid_link"/>
   </joint>
-  <xacro:web_camera camera_joint_type="$(arg camera_joint_type)" camera_pitch="$(arg camera_pitch)"
+  <xacro:web_camera tf_prefix="${tf_prefix}" camera_joint_type="$(arg camera_joint_type)" camera_pitch="$(arg camera_pitch)"
     camera_is_on="$(arg camera_is_on)"/>
 </robot>

Commit message: Updated URDF. Added sim launch file

File: thymioid_description/urdf/camera.urdf.xacro (robot description, xacro)
@@ -1,5 +1,5 @@
 <?xml version="1.0"?>
 <robot xmlns:xacro="http://playerstage.sourceforge.net/gazebo/xmlschema/#xacro">
-  <xacro:macro name="web_camera" params="tf_prefix='' camera_joint_type='fixed' camera_pitch=0">
+  <xacro:macro name="web_camera" params="ns='' tf_prefix='' camera_joint_type='fixed' camera_pitch=0">
     <link name="${tf_prefix}camera_support_link">
       <inertial>
@@ -103,4 +103,5 @@
           <frame_name>${tf_prefix}camera_optical_link</frame_name>
           <hack_baseline>0.0</hack_baseline>
+          <namespace>${ns}</namespace>
         </plugin>
       </sensor>

File: thymioid_description/urdf/thymioid.urdf.xacro (robot description, xacro)
@@ -123,4 +123,4 @@
     <child link="${tf_prefix}odroid_link"/>
   </joint>
-  <xacro:web_camera tf_prefix="${tf_prefix}" camera_joint_type="$(arg camera_joint_type)" camera_pitch="$(arg camera_pitch)"/>
+  <xacro:web_camera ns="${_name}" tf_prefix="${tf_prefix}" camera_joint_type="$(arg camera_joint_type)" camera_pitch="$(arg camera_pitch)"/>
 </robot>
